File: hardware/LPC43xx_blinky_board.sch (KiCad schematic (older format))
At the start: 43 parts

Commit message: Add Spifi Flash to lib and schematics
Parts:
- added C?: 100nF, symbol Device:C_Small
- added U?: SST26VF032B, Package_SO:SOIC-8_3.9x4.9mm_P1.27mm, symbol JitterLib:SST26VF032B
Connections:
- net labels added: SPIFI_CS, SPIFI_MISO, SPIFI_MOSI, SPIFI_SCK, SPIFI_SIO2, SPIFI_SIO3
- wire segments 113 -> 127
Other:
- note added: "== Spifi Flash =="
Changed lines of the file:
@@
 EESchema Schematic File Version 4
+LIBS:LPC43xx_blinky_board-cache
 EELAYER 26 0
 EELAYER END
@@
 	1    0    0    -1
 $EndComp
+$Comp
+L JitterLib:SST26VF032B U?
+U 1 1 5BA95B3D
+P 9050 5350
+F 0 "U?" H 8750 5800 50  0000 C CNN
+F 1 "SST26VF032B" H 8850 5000 50  0000 C CNN
+F 2 "Package_SO:SOIC-8_3.9x4.9mm_P1.27mm" H 8600 6150 50  0001 C CNN
+F 3 "http://www.farnell.com/datasheets/2245044.pdf" H 8750 6250 50  0001 C CNN
+	1    9050 5350
+	1    0    0    -1
+$EndComp
+Text Notes 8000 4300 0    118  ~ 24
+== Spifi Flash ==
+$Comp
+L power:GND #PWR?
+U 1 1 5BA97034
+P 9200 5750
+F 0 "#PWR?" H 9200 5500 50  0001 C CNN
+F 1 "GND" H 9205 5577 50  0000 C CNN
+F 2 "" H 9200 5750 50  0001 C CNN
+F 3 "" H 9200 5750 50  0001 C CNN
+	1    9200 5750
+	1    0    0    -1
+$EndComp
+$Comp
+L power:+3V3 #PWR?
+U 1 1 5BA97097
+P 9200 4700
+F 0 "#PWR?" H 9200 4550 50  0001 C CNN
+F 1 "+3V3" H 9215 4873 50  0000 C CNN
+F 2 "" H 9200 4700 50  0001 C CNN
+F 3 "" H 9200 4700 50  0001 C CNN
+	1    9200 4700
+	1    0    0    -1
+$EndComp
+Text Label 4050 9400 0    50   ~ 0
+SPIFI_SCK
+Text Label 4050 9500 0    50   ~ 0
+SPIFI_SIO3
+Text Label 4050 9600 0    50   ~ 0
+SPIFI_SIO2
+Text Label 4050 9700 0    50   ~ 0
+SPIFI_MISO
+Wire Wire Line
+	4050 9400 3950 9400
+Wire Wire Line
+	3950 9500 4050 9500
+Wire Wire Line
+	4050 9600 3950 9600
+Text Label 4050 9800 0    50   ~ 0
+SPIFI_MOSI
+Wire Wire Line
+	3950 9700 4050 9700
+Wire Wire Line
+	3950 9800 4050 9800
+Text Label 4050 9900 0    50   ~ 0
+SPIFI_CS
+Wire Wire Line
+	4050 9900 3950 9900
+Text Label 9650 5350 0    50   ~ 0
+SPIFI_SCK
+Text Label 7950 5450 0    50   ~ 0
+SPIFI_SIO3
+Text Label 7950 5350 0    50   ~ 0
+SPIFI_SIO2
+Text Label 7950 5250 0    50   ~ 0
+SPIFI_MISO
+Wire Wire Line
+	9650 5350 9550 5350
+Text Label 7950 5150 0    50   ~ 0
+SPIFI_MOSI
+Text Label 9650 5450 0    50   ~ 0
+SPIFI_CS
+Wire Wire Line
+	9650 5450 9550 5450
+Wire Wire Line
+	8600 5450 7950 5450
+Wire Wire Line
+	7950 5150 8600 5150
+Wire Wire Line
+	7950 5250 8600 5250
+Wire Wire Line
+	7950 5350 8600 5350
+$Comp
+L Device:C_Small C?
+U 1 1 5BAF7B28
+P 9700 4800
+F 0 "C?" H 9800 4950 50  0000 L CNN
+F 1 "100nF" H 9800 4850 50  0000 L CNN
+F 2 "" H 9700 4800 50  0001 C CNN
+F 3 "~" H 9700 4800 50  0001 C CNN
+	1    9700 4800
+	1    0    0    -1
+$EndComp
+$Comp
+L power:GND #PWR?
+U 1 1 5BAF7C82
+P 9700 4900
+F 0 "#PWR?" H 9700 4650 50  0001 C CNN
+F 1 "GND" H 9705 4727 50  0000 C CNN
+F 2 "" H 9700 4900 50  0001 C CNN
+F 3 "" H 9700 4900 50  0001 C CNN
+	1    9700 4900
+	1    0    0    -1
+$EndComp
+Wire Wire Line
+	9700 4700 9200 4700
+Wire Wire Line
+	9200 4700 9200 4950
+Connection ~ 9200 4700
 $EndSCHEMATC

Commit message: Add status leds and SD Card
Parts:
- removed C? (x16): 100nF, symbol Device:C_Small
- added C? (x14): 100nF, Capacitor_SMD:C_0402_1005Metric, symbol Device:C_Small
- added C? (x3): 100nF, Capacitor_SMD:C_0402_1005Metric, symbol Device:C
- added C?: 2.2nF, Capacitor_SMD:C_0402_1005Metric, symbol Device:C
- added D?: RED, symbol Device:LED
- added D?: GREEN, symbol Device:LED
- added D?: BLUE, symbol Device:LED
- added D?: YELLOW, symbol Device:LED
- added J?: Micro_SD_Card, symbol Connector:Micro_SD_Card
- added RN?: 220R, Resistor_SMD:R_Array_Convex_4x0402, symbol Device:R_Pack04
- C?: footprint (none) -> Capacitor_SMD:C_0402_1005Metric
Connections:
- net labels added: LED_BLUE, LED_GREEN, LED_RED, LED_YELLOW, SD_CLK, SD_CMD, SD_DAT0, SD_DAT1, SD_DAT2, SD_DAT3
- wire segments 127 -> 174
Other:
- note added: "== SD Card Slot =="
- note added: "== Status LEDs =="
- note added: "=== LPC43xx (4 parts) ==="
- note added: "— Decoupling —"
- note added: "— Essentials: Power, Debug, Crystal —"
- note added: "— Muliplexable pins 1/2 —"
- note added: "— Muliplexable pins 2/2 —"
- note added: "— USB, RTC, ADC, I2C —"
- note removed: "== Decoupling =="
- note removed: "== Essentials: Power, Debug, Crystal =="
- note removed: "== Miscellaneous =="
- note removed: "== USB, RTC, ADC, I2C =="

Commit message: Add headers with some selected useful pins to schematics
During routing pinswapping might still be desirable.
Parts:
- added C27: 10uF, Capacitor_SMD:C_0805_2012Metric, symbol Device:C
- added C28: 4.7uF, Capacitor_SMD:C_0805_2012Metric, symbol Device:C
- added C3, C4: 15pF, Capacitor_SMD:C_0402_1005Metric, symbol Device:C_Small
- added J2: USB_B_Micro, Connector_USB:USB_Micro-B_Molex_47346-0001, symbol Connector:USB_B_Micro
- added J4: Conn_01x20_Female, Connector_PinSocket_2.54mm:PinSocket_1x20_P2.54mm_Vertical, symbol Connector:Conn_01x20_Female
- added R2: 12k, Resistor_SMD:R_0402_1005Metric, symbol Device:R
- added U3: MCP1825S, Package_TO_SOT_SMD:SOT-223-3_TabPin2, symbol Regulator_Linear:MCP1825S
- added Y1: 32.768KHz, symbol Device:Crystal_Small
- D1, D2, D3, D4: renamed from D?; footprint (none) -> LED_SMD:LED_0603_1608Metric
- J3: renamed from J?; footprint (none) -> Connector_Card:microSD_HC_Wuerth_693072010801
- Y2: renamed from Y?; value Crystal -> 12MHz
- gave numbers to parts that had none: 44
Connections:
- net labels added: AD0, AD1, ALARM, CAN_RD, CAN_TD, CLKIN, SCL, SDA, TRACECLK, TRACEDATA0, TRACEDATA1, TRACEDATA2, TRACEDATA3, UART_RX, UART_TX, USB_HS_D+, USB_HS_D-, VBUS, WAKUP
- wire segments 174 -> 242
- no-connect marks 0 -> 74
Other:
- note added: "== IO Headers =="
- note added: "== LDO =="
- note added: "== USB =="

Commit message: All footprints are assigned. Ready for layout.
Parts:
- L1: value Ferrite_Bead -> 600 Ohm; footprint (none) -> Resistor_SMD:R_0402_1005Metric
- L2: value Ferrite_Bead -> 600 Ohm; footprint (none) -> Resistor_SMD:R_0402_1005Metric; Manufacturer PartNo. (none) -> BLM15HG601SN1D
- SW1: footprint (none) -> Button_Switch_SMD:SW_DIP_SPSTx01_Slide_Omron_A6S-110x_W8.9mm_P2.54mm
- SW3, SW4: footprint (none) -> Button_Switch_SMD:SW_SPST_EVQPE1
- Y1: footprint (none) -> misc:Crystal_SMD_Abracon_ABS07-2Pin_3.6x1.9mm
- Y2: footprint (none) -> Crystal:Crystal_SMD_TXC_7A-2Pin_5.0x3.2mm
Changed lines of the file:
@@
 F 0 "Y2" V 1746 5919 50  0000 R CNN
 F 1 "12MHz" V 1655 5919 50  0000 R CNN
-F 2 "" H 1700 6050 50  0001 C CNN
+F 2 "Crystal:Crystal_SMD_TXC_7A-2Pin_5.0x3.2mm" H 1700 6050 50  0001 C CNN
 F 3 "~" H 1700 6050 50  0001 C CNN
 	1    1700 6050
@@
 F 0 "SW1" H 13500 2467 50  0000 C CNN
 F 1 "SW_DIP_x01" H 13500 2376 50  0000 C CNN
-F 2 "" H 13500 2200 50  0001 C CNN
+F 2 "Button_Switch_SMD:SW_DIP_SPSTx01_Slide_Omron_A6S-110x_W8.9mm_P2.54mm" H 13500 2200 50  0001 C CNN
 F 3 "" H 13500 2200 50  0001 C CNN
 	1    13500 2200
@@
 P 9050 1550
 F 0 "L1" V 9100 1650 50  0000 C CNN
-F 1 "Ferrite_Bead" V 8950 1300 50  0000 C CNN
-F 2 "" V 8980 1550 50  0001 C CNN
-F 3 "~" H 9050 1550 50  0001 C CNN
+F 1 "600 Ohm" V 8950 1300 50  0000 C CNN
+F 2 "Resistor_SMD:R_0402_1005Metric" V 8980 1550 50  0001 C CNN
+F 3 "http://www.farnell.com/datasheets/5168.pdf" H 9050 1550 50  0001 C CNN
 	1    9050 1550
 	0    -1   -1   0
@@
 P 9150 5100
 F 0 "L2" V 9300 5150 50  0000 C CNN
-F 1 "Ferrite_Bead" V 9250 4750 50  0000 C CNN
-F 2 "" V 9080 5100 50  0001 C CNN
-F 3 "~" H 9150 5100 50  0001 C CNN
+F 1 "600 Ohm" V 9250 4750 50  0000 C CNN
+F 2 "Resistor_SMD:R_0402_1005Metric" V 9080 5100 50  0001 C CNN
+F 3 "http://www.farnell.com/datasheets/5168.pdf" H 9150 5100 50  0001 C CNN
+F 4 "BLM15HG601SN1D" V 9150 5100 50  0001 C CNN "Manufacturer PartNo."
 	1    9150 5100
 	0    -1   -1   0
@@
 F 0 "SW3" H 4000 9285 50  0000 C CNN
 F 1 "SW_SPST" H 4000 9194 50  0000 C CNN
-F 2 "" H 4000 9050 50  0001 C CNN
+F 2 "Button_Switch_SMD:SW_SPST_EVQPE1" H 4000 9050 50  0001 C CNN
 F 3 "" H 4000 9050 50  0001 C CNN
 	1    4000 9050
@@
 F 0 "SW4" H 5650 9285 50  0000 C CNN
 F 1 "SW_SPST" H 5650 9194 50  0000 C CNN
-F 2 "" H 5650 9050 50  0001 C CNN
+F 2 "Button_Switch_SMD:SW_SPST_EVQPE1" H 5650 9050 50  0001 C CNN
 F 3 "" H 5650 9050 50  0001 C CNN
 	1    5650 9050
@@
 F 0 "Y1" V 10150 2300 50  0000 L CNN
 F 1 "32.768KHz" V 10000 2250 50  0000 L CNN
-F 2 "" H 10150 2550 50  0001 C CNN
+F 2 "misc:Crystal_SMD_Abracon_ABS07-2Pin_3.6x1.9mm" H 10150 2550 50  0001 C CNN
 F 3 "~" H 10150 2550 50  0001 C CNN
 	1    10150 2550

Commit message: Starting layout work for blinky board
Parts:
- added J5: Conn_01x04_Male, Connector_PinHeader_2.54mm:PinHeader_1x04_P2.54mm_Horizontal, symbol Connector:Conn_01x04_Male
Connections:
- net labels added: SWDCLK, SWDIO
- wire segments 242 -> 246
Other:
- note added: "== Extra SWD Header =="
Changed lines of the file:
@@
 F 3 "~" H 1700 6050 50  0001 C CNN
 	1    1700 6050
-	0    -1   -1   0
+	0    1    1    0
 $EndComp
 Wire Wire Line
@@
 	9000 5100 8950 5100
 Connection ~ 8950 5100
+$Comp
+L Connector:Conn_01x04_Male J5
+U 1 1 5BACCD71
+P 14850 5700
+F 0 "J5" H 14956 5978 50  0000 C CNN
+F 1 "Conn_01x04_Male" H 14956 5887 50  0000 C CNN
+F 2 "Connector_PinHeader_2.54mm:PinHeader_1x04_P2.54mm_Horizontal" H 14850 5700 50  0001 C CNN
+F 3 "~" H 14850 5700 50  0001 C CNN
+	1    14850 5700
+	1    0    0    -1
+$EndComp
+Text Label 4200 6200 0    50   ~ 0
+SWDCLK
+Text Label 4200 6300 0    50   ~ 0
+SWDIO
+$Comp
+L power:+3V3 #PWR01
+U 1 1 5BACEA4B
+P 15400 5600
+F 0 "#PWR01" H 15400 5450 50  0001 C CNN
+F 1 "+3V3" H 15415 5773 50  0000 C CNN
+F 2 "" H 15400 5600 50  0001 C CNN
+F 3 "" H 15400 5600 50  0001 C CNN
+	1    15400 5600
+	1    0    0    -1
+$EndComp
+Wire Wire Line
+	15050 5600 15400 5600
+$Comp
+L power:GND #PWR02
+U 1 1 5BAE2549
+P 15400 5900
+F 0 "#PWR02" H 15400 5650 50  0001 C CNN
+F 1 "GND" H 15405 5727 50  0000 C CNN
+F 2 "" H 15400 5900 50  0001 C CNN
+F 3 "" H 15400 5900 50  0001 C CNN
+	1    15400 5900
+	1    0    0    -1
+$EndComp
+Wire Wire Line
+	15050 5900 15400 5900
+Text Label 15150 5800 0    50   ~ 0
+SWDCLK
+Wire Wire Line
+	15050 5800 15150 5800
+Text Label 15150 5700 0    50   ~ 0
+SWDIO
+Wire Wire Line
+	15050 5700 15150 5700
+Text Notes 14350 5250 0    79   ~ 16
+== Extra SWD Header ==
 $EndSCHEMATC

Commit message: Routed the left side of the board
- USB
- JTAG
- Crystals
Connections:
- net labels added: USB_ID
- wire segments 246 -> 250
- no-connect marks 74 -> 68
Changed lines of the file:
@@
 	11050 7650 500  7650
 NoConn ~ 9800 3750
-NoConn ~ 9800 4050
 NoConn ~ 9800 4350
 NoConn ~ 9800 4450
@@
 Wire Wire Line
 	15350 8800 14750 8800
-NoConn ~ 12450 7450
 NoConn ~ 15350 8000
 NoConn ~ 15350 7700
@@
 	7000 2050 6700 2050
 Wire Wire Line
-	7000 1950 6700 1950
-Wire Wire Line
-	7000 1850 6700 1850
+	3400 2950 3300 2950
+Wire Wire Line
+	3400 2850 3300 2850
 Wire Wire Line
 	7000 1750 6700 1750
-Text Label 7000 2050 0    50   ~ 0
+Text Label 3400 3050 0    50   ~ 0
 LED_RED
-Text Label 7000 1950 0    50   ~ 0
+Text Label 3400 2950 0    50   ~ 0
 LED_GREEN
-Text Label 7000 1850 0    50   ~ 0
+Text Label 3400 2850 0    50   ~ 0
 LED_BLUE
-Text Label 7000 1750 0    50   ~ 0
+Text Label 3400 2750 0    50   ~ 0
 LED_YELLOW
 Text Label 7000 2150 0    50   ~ 0
@@
 NoConn ~ 1400 3650
 NoConn ~ 3300 3250
-NoConn ~ 3300 3050
-NoConn ~ 3300 2850
-NoConn ~ 3300 2750
-NoConn ~ 3300 2950
 NoConn ~ 3300 2350
 NoConn ~ 3300 2250
@@
 Text Notes 14350 5250 0    79   ~ 16
 == Extra SWD Header ==
+Wire Wire Line
+	3300 3050 3400 3050
+Wire Wire Line
+	3300 2750 3400 2750
+Text Label 9950 4050 0    50   ~ 0
+USB_ID
+Wire Wire Line
+	9800 4050 9950 4050
+Text Label 11800 7450 0    50   ~ 0
+USB_ID
+Wire Wire Line
+	11800 7450 12450 7450
 $EndSCHEMATC

Commit message: Finish routing except random IO headers
Parts:
- removed C29: 100nF, Capacitor_SMD:C_0402_1005Metric, symbol Device:C
- removed R6: 100k, Resistor_SMD:R_0402_1005Metric, symbol Device:R
- added J6: Conn_01x04_Female, Connector_PinSocket_2.54mm:PinSocket_1x04_P2.54mm_Vertical, symbol Connector:Conn_01x04_Female
- added J7: Conn_01x08_Female, Connector_PinSocket_2.54mm:PinSocket_1x08_P2.54mm_Vertical, symbol Connector:Conn_01x08_Female
- J4: footprint Connector_PinSocket_2.54mm:PinSocket_1x20_P2.54mm_Vertical -> Connector_PinSocket_2.54mm:PinSocket_1x10_P2.54mm_Vertical; symbol Connector:Conn_01x20_Female -> Connector:Conn_01x10_Female
- renumbered C30 to C29, J5 to J1, J1 to J2, J2 to J3, J3 to J5, R7 to R6
Connections:
- wire segments 250 -> 251
- no-connect marks 68 -> 72
Other:
- note added: "Pullup and cap already in jtag section"

Commit message: Route all missing connections
Connections:
- wire segments 251 -> 253
- no-connect marks 72 -> 68
Changed lines of the file:
@@
 Wire Wire Line
 	3300 3450 3400 3450
-Text Label 14350 1600 0    50   ~ 0
+Text Label 14000 9450 0    50   ~ 0
 CAN_TD
-Text Label 14350 1500 0    50   ~ 0
+Text Label 14000 9550 0    50   ~ 0
 CAN_RD
 Text Notes 14250 6650 0    118  ~ 24
@@
 Wire Wire Line
 	4450 2450 4800 2450
-Text Label 14750 8600 0    50   ~ 0
+Text Label 14000 9150 0    50   ~ 0
 CLKIN
-Text Label 14350 1900 0    50   ~ 0
+Text Label 14000 7400 0    50   ~ 0
 UART_TX
-Text Label 14350 2000 0    50   ~ 0
+Text Label 14000 7500 0    50   ~ 0
 UART_RX
 Text Label 7550 3950 0    50   ~ 0
@@
 Wire Wire Line
 	6700 3850 6900 3850
-Text Label 14750 8500 0    50   ~ 0
+Text Label 14000 9050 0    50   ~ 0
 TRACECLK
-Text Label 14750 8100 0    50   ~ 0
+Text Label 14000 8950 0    50   ~ 0
 TRACEDATA0
-Text Label 14750 8200 0    50   ~ 0
+Text Label 14000 8850 0    50   ~ 0
 TRACEDATA1
-Text Label 14750 8300 0    50   ~ 0
+Text Label 14000 8750 0    50   ~ 0
 TRACEDATA2
-Text Label 14750 8400 0    50   ~ 0
+Text Label 14000 8650 0    50   ~ 0
 TRACEDATA3
 Wire Notes Line
@@
 Wire Wire Line
 	9800 2900 10000 2900
-Text Label 14750 8800 0    50   ~ 0
+Text Label 14000 9250 0    50   ~ 0
 WAKUP
-Text Label 14750 8700 0    50   ~ 0
+Text Label 14000 9350 0    50   ~ 0
 ALARM
-Text Label 14350 2100 0    50   ~ 0
+Text Label 14000 8000 0    50   ~ 0
 AD0
-Text Label 14350 2200 0    50   ~ 0
+Text Label 14000 8100 0    50   ~ 0
 AD1
 $Comp
 L Connector:Conn_01x10_Female J4
 U 1 1 5C2D4F1D
-P 15550 8000
-F 0 "J4" H 14600 6850 50  0000 L CNN
-F 1 "Conn_01x20_Female" H 14800 6850 50  0000 L CNN
-F 2 "Connector_PinSocket_2.54mm:PinSocket_1x10_P2.54mm_Vertical" H 15550 8000 50  0001 C CNN
-F 3 "~" H 15550 8000 50  0001 C CNN
-	1    15550 8000
-	1    0    0    -1
-$EndComp
-Wire Wire Line
-	14950 1500 14350 1500
-Wire Wire Line
-	14350 1600 14950 1600
-Wire Wire Line
-	14350 1900 14950 1900
-Wire Wire Line
-	14950 2000 14350 2000
-Wire Wire Line
-	14350 2100 14950 2100
-Wire Wire Line
-	14950 2200 14350 2200
-Wire Wire Line
-	14750 8100 15350 8100
-Wire Wire Line
-	15350 8200 14750 8200
-Wire Wire Line
-	14750 8300 15350 8300
-Wire Wire Line
-	15350 8400 14750 8400
-Wire Wire Line
-	14750 8600 15350 8600
-Wire Wire Line
-	14750 8500 15350 8500
-Wire Wire Line
-	14750 8700 15350 8700
-Wire Wire Line
-	15350 8800 14750 8800
-NoConn ~ 15350 8000
-NoConn ~ 15350 7700
-NoConn ~ 15350 7400
-NoConn ~ 15350 7300
-Text Label 14750 8900 0    50   ~ 0
+P 14800 9050
+F 0 "J4" H 13950 8400 50  0000 L CNN
+F 1 "Conn_01x20_Female" H 14100 8400 50  0000 L CNN
+F 2 "Connector_PinSocket_2.54mm:PinSocket_1x10_P2.54mm_Vertical" H 14800 9050 50  0001 C CNN
+F 3 "~" H 14800 9050 50  0001 C CNN
+	1    14800 9050
+	1    0    0    -1
+$EndComp
+Wire Wire Line
+	14600 7400 14000 7400
+Wire Wire Line
+	14000 7500 14600 7500
+Wire Wire Line
+	14000 7800 14600 7800
+Wire Wire Line
+	14600 7900 14000 7900
+Wire Wire Line
+	14000 8000 14600 8000
+Wire Wire Line
+	14600 8100 14000 8100
+Wire Wire Line
+	14000 8650 14600 8650
+Wire Wire Line
+	14600 8750 14000 8750
+Wire Wire Line
+	14000 8850 14600 8850
+Wire Wire Line
+	14600 8950 14000 8950
+Wire Wire Line
+	14000 9150 14600 9150
+Wire Wire Line
+	14000 9050 14600 9050
+Wire Wire Line
+	14000 9250 14600 9250
+Wire Wire Line
+	14600 9350 14000 9350
+Text Label 14000 7700 0    50   ~ 0
 SDA
-Text Label 14750 9000 0    50   ~ 0
+Text Label 14000 7600 0    50   ~ 0
 SCL
 Wire Wire Line
-	14750 8900 15350 8900
-Wire Wire Line
-	14750 9000 15350 9000
+	14000 9450 14600 9450
+Wire Wire Line
+	14000 9550 14600 9550
 Wire Wire Line
 	14250 3650 14150 3650
@@
 L Connector:Conn_01x08_Female J7
 U 1 1 5BD58EF6
-P 15150 1800
-F 0 "J7" H 15177 1776 50  0000 L CNN
-F 1 "Conn_01x08_Female" H 15177 1685 50  0000 L CNN
-F 2 "Connector_PinSocket_2.54mm:PinSocket_1x08_P2.54mm_Vertical" H 15150 1800 50  0001 C CNN
-F 3 "~" H 15150 1800 50  0001 C CNN
-	1    15150 1800
-	1    0    0    -1
-$EndComp
+P 14800 7700
+F 0 "J7" H 14827 7676 50  0000 L CNN
+F 1 "Conn_01x08_Female" H 14827 7585 50  0000 L CNN
+F 2 "Connector_PinSocket_2.54mm:PinSocket_1x08_P2.54mm_Vertical" H 14800 7700 50  0001 C CNN
+F 3 "~" H 14800 7700 50  0001 C CNN
+	1    14800 7700
+	1    0    0    -1
+$EndComp
+Wire Wire Line
+	14000 7600 14600 7600
+Wire Wire Line
+	14000 7700 14600 7700
 $EndSCHEMATC
